File: left_hand/hecomi.sch (KiCad schematic (older format))
At the start: 75 parts, among them J1 Conn_01x03_Female, J2 Conn_01x04_Female, J3 Conn_01x04_Female, SW1 SW_Push, SW10 SW_Push, SW11 SW_Push, SW12 SW_Push, SW13 SW_Push, SW14 SW_Push, SW15 SW_Push, SW16 SW_Push, SW17 SW_Push, SW18 SW_Push, SW19 SW_Push, SW2 SW_Push, SW20 SW_Push, SW21 SW_Push, SW22 SW_Push, SW23 SW_Push, SW24 SW_Push, SW25 SW_Push, SW26 SW_Push, SW27 SW_Push, SW28 SW_Push, SW29 SW_Push, SW3 SW_Push, SW30 SW_Push, SW31 SW_Push, SW32 SW_Push, SW33 SW_Push, SW34 SW_Push, SW35 SW_Push, SW36 SW_Push, SW4 SW_Push, SW5 SW_Push, SW6 SW_Push, SW7 SW_Push, SW8 SW_Push, SW9 SW_Push, U1 ProMicro

Commit message: end
Parts:
- added J4: Conn_01x07_Female, My_Keyboard:usb_type-c_akitsuki, symbol Connector:Conn_01x07_Female
- added J5: Conn_01x04_Female, Connector_PinSocket_2.54mm:PinSocket_1x04_P2.54mm_Vertical, symbol Connector:Conn_01x04_Female
- added MH1, MH10, MH2, MH3, MH4, MH5, MH6, MH7, MH8, MH9: MountingHole, My_Keyboard:MountingHole_2.2mm_M2, symbol Mechanical:MountingHole
- J2, J3: footprint Connector_PinHeader_2.54mm:PinHeader_1x04_P2.54mm_Vertical -> Keebio-Parts:TRRS-PJ-320A
- SW1, SW10, SW11, SW12, SW13, SW14, SW15, SW16, SW17, SW18, SW19, SW2, SW20, SW21, SW22, SW23, SW24, SW25, SW26, SW27, SW28, SW29, SW3, SW30, SW31, SW32, SW33, SW34, SW35, SW4, SW5, SW6, SW7, SW8, SW9: footprint (none) -> My_Keyboard:MXOnly-1U-Hotswap-Antishear
- SW36: footprint (none) -> My_Keyboard:1101VS-E
- U1: footprint (none) -> My_Keyboard:ProMicro
Connections:
- net labels added: D+, D-, VBUS
- no-connect marks 1 -> 4
